File: KiCad/V1/GameboyCartridgeV1.1/GameboyCartridgeV1.1.kicad_pcb (KiCad board)
At the start: 4 copper layers, 52.8 x 61.2 mm, 56 parts, among them J1 USB_C_Receptacle_USB2.0, J2 DBG_UART, J3 Conn_01x06, Q1 CJ2302, SW1 SW_Push, U1 W25Q128JVS, U2 RP2040, U3 CartBus, U4 MCP1825T-3302E/DC, U5 TXB0102DCU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

Commit message: main changes
Parts:
- removed C16: 10uF, Capacitor_SMD:C_0603_1608Metric_Pad1.08x0.95mm_HandSolder
- removed U4: MCP1825T-3302E/DC, SnapEDA:SOT230P700X180-6N
- added C25: 1µF, Capacitor_SMD:C_0603_1608Metric_Pad1.08x0.95mm_HandSolder, F.Cu at (92.0, 77.5)
- added C26: 1µF, Capacitor_SMD:C_0603_1608Metric_Pad1.08x0.95mm_HandSolder, F.Cu at (98.0, 77.5)
- added C27: 22µF, Capacitor_SMD:C_0805_2012Metric, F.Cu at (97.2, 80.5)
- added U9: RT9080, Package_TO_SOT_SMD:SOT-23-5, F.Cu at (95.0, 77.5)
- C10, C12, C13, C2, C5, C6, C8, C9: footprint Capacitor_SMD:C_0402_1005Metric_Pad0.74x0.62mm_HandSolder -> Capacitor_SMD:C_0603_1608Metric_Pad1.08x0.95mm_HandSolder
- C15: value 4.7uF -> 1µF
- D1: footprint LED_SMD:LED_WS2812B_PLCC4_5.0x5.0mm_P3.2mm -> LED_SMD:LED_WS2812B-2020_PLCC4_2.0x2.0mm
- D2, D3: footprint Diode_SMD:D_SOD-123F -> Diode_SMD:D_SOD-323
- R7: value 470k -> 10k
- SW1: footprint Button_Switch_SMD:SW_SPST_TL3342 -> Button_Switch_SMD:SW_Push_SPST_NO_Alps_SKRK
- moved R7 5.25 mm to (93.4, 81.8), turned to 0 degrees
- moved C15 3.81 mm to (93.4, 83.2)
- moved C14 2.88 mm to (104.0, 61.0)
- moved C9 1.56 mm to (114.5, 87.2), turned to -90 degrees
- moved C2 0.83 mm to (112.8, 73.8)
- moved C12 0.76 mm to (111.2, 73.8)
- moved C13 0.62 mm to (116.0, 87.2), turned to -90 degrees
- moved C3 0.55 mm to (108.8, 93.2)
- moved C4 0.50 mm to (113.8, 93.2)
- moved R2 0.45 mm to (114.2, 73.8)
- moved C11 0.25 mm to (118.8, 73.8)
- moved C7 0.25 mm to (117.2, 73.8)
- moved R3 0.25 mm to (115.8, 73.8)
- moved SW1 0.17 mm to (127.8, 72.5)
- moved C5 0.16 mm to (119.0, 81.8)
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Connections:
- C15 pad 2: +5V -> POWER_GOOD
- R7 pad 1: POWER_GOOD -> +3V3
- R7 pad 2: +3V3 -> POWER_GOOD
Routing:
- net VCC: track 35.3 -> 83.9 mm, vias 5 -> 4
- net +3V3: track 72.9 -> 96.9 mm, vias 19 -> 11
- net GND: track 68.5 -> 58.8 mm, vias 192 -> 158
- net RST: track 54.5 -> 48.2 mm
- net +5V: track 18.3 -> 24.0 mm
- net USB_D-: track 13.4 -> 18.4 mm, vias 0 -> 2
- net +1V1: track 23.6 -> 21.2 mm, vias 3 -> 4
- net POWER_GOOD: track 76.5 -> 74.4 mm
- net USB_D+: track 12.2 -> 14.0 mm
- net LED_DIN: track 46.9 -> 48.4 mm
- net DATA_BUS3: track 29.9 -> 28.6 mm
- net DATA_BUS2: track 28.9 -> 27.7 mm
- net DATA_BUS1: track 27.9 -> 26.8 mm
- net DATA_BUS0: track 26.9 -> 26.0 mm
- net SWDIO: track 18.0 -> 17.1 mm
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- added copper zone on F.Cu, net +1V1
- added copper zone on F.Cu, net +3V3
- added copper zone on F.Cu, net GND
- added copper zone on F.Cu, net VBUS
- removed copper zone on In2.Cu, net +3V3
- removed copper zone on In1.Cu, net GND
- removed copper zone on In2.Cu, net VBUS
- removed copper zone on In2.Cu, net VCC
Other:
- copper layers 4 -> 2
