File: KiCad/V1/GameboyCartridgeV1.1/power.kicad_sch (KiCad schematic)
At the start: 25 parts, among them Q1 CJ2302, U3 CartBus, U4 MCP1825T-3302E/DC, U5 TXB0102DCU, U6 TXB0108PW, U7 TXB0108PW, U8 TXB0108PW

Commit message: main changes
Parts:
- removed C15: 4.7uF, Capacitor_SMD:C_0603_1608Metric_Pad1.08x0.95mm_HandSolder, symbol Device:C
- removed C16: 10uF, Capacitor_SMD:C_0603_1608Metric_Pad1.08x0.95mm_HandSolder, symbol Device:C
- removed U4: MCP1825T-3302E/DC, SnapEDA:SOT230P700X180-6N, symbol MCP1825T-3302E_DC:MCP1825T-3302E/DC
- added C15, C25, C26: 1µF, Capacitor_SMD:C_0603_1608Metric_Pad1.08x0.95mm_HandSolder, symbol Device:C_Small
- added C27: 22µF, Capacitor_SMD:C_0805_2012Metric, symbol Device:C_Small
- added U9: RT9080, Package_TO_SOT_SMD:SOT-23-5, symbol Regulator_Linear:TLV75533PDBV
- D2, D3: footprint Diode_SMD:D_SOD-123F -> Diode_SMD:D_SOD-323
- R7: value 470k -> 10k
Connections:
- net +3V3: now also R7.1, C26.2, C27.2, U9.5 (OUT); no longer R7.2
- net +5V: now also C25.2, U9.1 (IN), U9.3 (EN)
- net GND: now also C15.1, C25.1, C26.1, C27.1, U9.2 (GND)
- net POWER_GOOD: now also R7.2, C15.2; no longer R7.1
Other:
- moved on the sheet: C18
